Commit message: [WIP] Add draft of 6D joint pose calibration.

File: talos_description/urdf/arm/arm.urdf.xacro (robot description, xacro)
@@ -28,4 +28,8 @@
     <!--        SHOULDER        -->
     <!--************************-->
+    <xacro:calibration_joint name="${name}_${side}_1" parent="${parent}">
+      <origin xyz="0.00000 ${0.15750*reflect} 0.23200"
+              rpy="${0.0 * deg_to_rad} ${0.0 * deg_to_rad} ${0.0 * deg_to_rad}"/>
+    </xacro:calibration_joint>
     <link name="${name}_${side}_1_link">
       <xacro:call macro="${name}_${side}_1_link_inertial" />
@@ -45,8 +49,7 @@
     </link>
     <joint name="${name}_${side}_1_joint" type="revolute">
-      <parent link="${parent}" />
+      <parent link="${name}_${side}_1_calibration_link" />
       <child link="${name}_${side}_1_link" />
-      <origin xyz="0.00000 ${0.15750*reflect} 0.23200"
-              rpy="${0.0 * deg_to_rad} ${0.0 * deg_to_rad} ${0.0 * deg_to_rad}"/>
+      <xacro:joint_offset which="${name}_${side}" id="1"/>
       <axis xyz="0 0 1" />
       <xacro:arm_1_joint_limits reflect="${reflect}" />

File: talos_description/urdf/talos_full_common.urdf.xacro (robot description, xacro)
@@ -22,4 +22,5 @@
   <xacro:include filename="$(find talos_description)/urdf/leg/foot_collision_$(arg foot_collision).urdf.xacro" />
   <xacro:include filename="$(find talos_description_inertial)/urdf/inertial.xacro" />
+  <xacro:include filename="$(find talos_description)/urdf/extras/calibration.urdf.xacro" />
   <xacro:include filename="$(find talos_description)/urdf/extras/addons.urdf.xacro" />
   <xacro:talos_torso name="torso" />

File: talos_description_calibration/urdf/calibration/calibration_constants.urdf.xacro (robot description, xacro)
@@ -40,3 +40,23 @@
   <xacro:property name="torso_imu_pitch_offset" value="0.0" />
   <xacro:property name="torso_imu_yaw_offset" value="0.0" />
+  <xacro:macro name="joint_offset" params="which id">
+    <xacro:if value="${which == 'arm_left'}">
+      <xacro:if value="${id == 1}"> <origin xyz="0 0 0" rpy="0 0 0"/> </xacro:if>
+      <xacro:if value="${id == 2}"> <origin xyz="0 0 0" rpy="0 0 0"/> </xacro:if>
+      <xacro:if value="${id == 3}"> <origin xyz="0 0 0" rpy="0 0 0"/> </xacro:if>
+      <xacro:if value="${id == 4}"> <origin xyz="0 0 0" rpy="0 0 0"/> </xacro:if>
+      <xacro:if value="${id == 5}"> <origin xyz="0 0 0" rpy="0 0 0"/> </xacro:if>
+      <xacro:if value="${id == 6}"> <origin xyz="0 0 0" rpy="0 0 0"/> </xacro:if>
+      <xacro:if value="${id == 7}"> <origin xyz="0 0 0" rpy="0 0 0"/> </xacro:if>
+    </xacro:if>
+    <xacro:if value="${which == 'arm_right'}">
+      <xacro:if value="${id == 1}"> <origin xyz="0 0 0" rpy="0 0 0"/> </xacro:if>
+      <xacro:if value="${id == 2}"> <origin xyz="0 0 0" rpy="0 0 0"/> </xacro:if>
+      <xacro:if value="${id == 3}"> <origin xyz="0 0 0" rpy="0 0 0"/> </xacro:if>
+      <xacro:if value="${id == 4}"> <origin xyz="0 0 0" rpy="0 0 0"/> </xacro:if>
+      <xacro:if value="${id == 5}"> <origin xyz="0 0 0" rpy="0 0 0"/> </xacro:if>
+      <xacro:if value="${id == 6}"> <origin xyz="0 0 0" rpy="0 0 0"/> </xacro:if>
+      <xacro:if value="${id == 7}"> <origin xyz="0 0 0" rpy="0 0 0"/> </xacro:if>
+    </xacro:if>
+  </xacro:macro>
 </robot>

Commit message: Enable 6D calibration of arm, head and torso joints.

File: talos_description/urdf/arm/arm.urdf.xacro (robot description, xacro)
@@ -25,4 +25,5 @@
   <xacro:property name="arm_eps"            value="0.02" />
   <xacro:macro name="talos_arm" params="name parent side reflect">
+    <xacro:include filename="$(find talos_description_calibration)/urdf/calibration/arm_${side}.xacro" />
     <!--************************-->
     <!--        SHOULDER        -->
@@ -47,6 +48,6 @@
       <parent link="${parent}" />
       <child link="${name}_${side}_1_link" />
-      <origin xyz="0.00000 ${0.15750*reflect} 0.23200"
-              rpy="${0.0 * deg_to_rad} ${0.0 * deg_to_rad} ${0.0 * deg_to_rad}"/>
+      <origin xyz="${0.00000 + arm_1_joint_x_offset} ${0.15750*reflect + arm_1_joint_y_offset} ${0.23200 + arm_1_joint_z_offset}"
+              rpy="${0.0 * deg_to_rad + arm_1_joint_roll_offset} ${0.0 * deg_to_rad + arm_1_joint_pitch_offset} ${0.0 * deg_to_rad + arm_1_joint_yaw_offset}"/>
       <axis xyz="0 0 1" />
       <xacro:arm_1_joint_limits reflect="${reflect}" />
@@ -76,6 +77,6 @@
       <parent link="${name}_${side}_1_link" />
       <child link="${name}_${side}_2_link" />
-      <origin xyz="0.00493 ${0.13650*reflect} 0.04673"
-              rpy="${0.00000 * deg_to_rad} ${0.00000 * deg_to_rad} ${0.00000 * deg_to_rad}"/>
+      <origin xyz="${0.00493 + arm_2_joint_x_offset} ${0.13650*reflect + arm_2_joint_y_offset} ${0.04673 + arm_2_joint_z_offset}"
+              rpy="${0.00000 * deg_to_rad + arm_2_joint_roll_offset} ${0.00000 * deg_to_rad + arm_2_joint_pitch_offset} ${0.00000 * deg_to_rad + arm_2_joint_yaw_offset}"/>
       <axis xyz="1 0 0" />
       <limit lower="${(-82.0000 + 82.5000*reflect)* deg_to_rad}" upper="${(82.50000*reflect + 82.0000)* deg_to_rad}" effort="${arm_2_max_effort}" velocity="${arm_2_max_vel}" />
@@ -105,6 +106,6 @@
       <parent link="${name}_${side}_2_link" />
       <child link="${name}_${side}_3_link" />
-      <origin xyz="0.00000 0.00000 0.00000"
-              rpy="${0.00000 * deg_to_rad} ${0.00000 * deg_to_rad} ${0.00000 * deg_to_rad}"/>
+      <origin xyz="${0.00000 + arm_3_joint_x_offset} ${0.00000 + arm_3_joint_y_offset} ${0.00000 + arm_3_joint_z_offset}"
+              rpy="${0.00000 * deg_to_rad + arm_3_joint_roll_offset} ${0.00000 * deg_to_rad + arm_3_joint_pitch_offset} ${0.00000 * deg_to_rad + arm_3_joint_yaw_offset}"/>
       <axis xyz="0 0 1" />
       <limit lower="${-139.0 * deg_to_rad}" upper="${139.0 * deg_to_rad}" effort="${arm_3_max_effort}" velocity="${arm_3_max_vel}" />
@@ -137,6 +138,6 @@
       <parent link="${name}_${side}_3_link" />
       <child link="${name}_${side}_4_link" />
-      <origin xyz="0.02000 0.00000 -0.27300"
-              rpy="${0.00000 * deg_to_rad} ${0.00000 * deg_to_rad} ${0.00000 * deg_to_rad}"/>
+      <origin xyz="${0.02000 + arm_4_joint_x_offset} ${0.00000 + arm_4_joint_y_offset} ${-0.27300 + arm_4_joint_z_offset}"
+              rpy="${0.00000 * deg_to_rad + arm_4_joint_roll_offset} ${0.00000 * deg_to_rad + arm_4_joint_pitch_offset} ${0.00000 * deg_to_rad + arm_4_joint_yaw_offset}"/>
       <axis xyz="0 1 0" />
       <limit lower="${-128.0 * deg_to_rad}" upper="${-0.2 * deg_to_rad}" effort="${arm_4_max_effort}" velocity="${arm_4_max_vel}" />

File: talos_description/urdf/arm/wrist.urdf.xacro (robot description, xacro)
@@ -22,4 +22,5 @@
   <xacro:property name="wrist_eps"          value="0.02" />
   <xacro:macro name="talos_wrist" params="name parent side reflect">
+    <xacro:include filename="$(find talos_description_calibration)/urdf/calibration/arm_${side}.xacro" />
     <!--************************-->
     <!--        WRIST           -->
@@ -44,6 +45,6 @@
       <parent link="${parent}" />
       <child link="${name}_${side}_5_link" />
-      <origin xyz="-0.02000 0.00000 -0.26430"
-                rpy="${0.00000 * deg_to_rad} ${0.00000 * deg_to_rad} ${0.00000 * deg_to_rad}"/>
+      <origin xyz="${-0.02000 + arm_5_joint_x_offset} ${0.00000 + arm_5_joint_y_offset} ${-0.26430 + arm_5_joint_z_offset}"
+              rpy="${0.00000 * deg_to_rad + arm_5_joint_roll_offset} ${0.00000 * deg_to_rad + arm_5_joint_pitch_offset} ${0.00000 * deg_to_rad + arm_5_joint_yaw_offset}"/>
       <axis xyz="0 0 1" />
       <limit lower="${-144.0 * deg_to_rad}" upper="${144.0 * deg_to_rad}" effort="${wrist_1_max_effort}" velocity="${wrist_1_max_vel}" />
@@ -73,6 +74,6 @@
       <parent link="${name}_${side}_5_link" />
       <child link="${name}_${side}_6_link" />
-      <origin xyz="0.00000 0.00000 0.00000"
-              rpy="${0.00000 * deg_to_rad} ${0.00000 * deg_to_rad} ${0.00000 * deg_to_rad}"/>
+      <origin xyz="${0.00000 + arm_6_joint_x_offset} ${0.00000 + arm_6_joint_y_offset} ${0.00000 + arm_6_joint_z_offset}"
+              rpy="${0.00000 * deg_to_rad + arm_6_joint_roll_offset} ${0.00000 * deg_to_rad + arm_6_joint_pitch_offset} ${0.00000 * deg_to_rad + arm_6_joint_yaw_offset}"/>
       <axis xyz="1 0 0" />
       <limit lower="${-78.5 * deg_to_rad}" upper="${78.5 * deg_to_rad}" effort="${wrist_2_max_effort}" velocity="${wrist_2_max_vel}" />
@@ -102,6 +103,6 @@
       <parent link="${name}_${side}_6_link" />
       <child link="${name}_${side}_7_link" />
-      <origin xyz="0.0 0.0 0.0"
-                rpy="${0.0 * deg_to_rad} ${0.0 * deg_to_rad} ${0.0 * deg_to_rad}"/>
+      <origin xyz="${0.00000 + arm_7_joint_x_offset} ${0.00000 + arm_7_joint_y_offset} ${0.00000 + arm_7_joint_z_offset}"
+              rpy="${0.00000 * deg_to_rad + arm_7_joint_roll_offset} ${0.00000 * deg_to_rad + arm_7_joint_pitch_offset} ${0.00000 * deg_to_rad + arm_7_joint_yaw_offset}"/>
       <axis xyz="0 1 0" />
       <limit lower="${-39.0 * deg_to_rad}" upper="${39.0 * deg_to_rad}" effort="${wrist_3_max_effort}" velocity="${wrist_3_max_vel}"/>

File: talos_description/urdf/head/head.urdf.xacro (robot description, xacro)
@@ -41,6 +41,6 @@
       <parent link="${parent}"/>
       <child link="${name}_link"/>
-      <origin xyz="0.02000 0.00000 0.32100"
-              rpy="${0.00000 * deg_to_rad} ${0.00000 * deg_to_rad} ${0.00000 * deg_to_rad}"/>
+      <origin xyz="${0.02000 + head_1_joint_x_offset} ${0.00000 + head_1_joint_y_offset} ${0.32100 + head_1_joint_z_offset}"
+              rpy="${0.00000 * deg_to_rad + head_1_joint_roll_offset} ${0.00000 * deg_to_rad + head_1_joint_pitch_offset} ${0.00000 * deg_to_rad + head_1_joint_yaw_offset}"/>
       <axis xyz="0 1 0" />
       <limit lower="${-12.00000 * deg_to_rad}" upper="${45.00000 * deg_to_rad}" effort="8.0" velocity="${head_max_vel}" />
@@ -85,6 +85,6 @@
       <parent link="${parent}"/>
       <child link="${name}_link"/>
-      <origin xyz="0.00000 0.00000 0.00000"
-              rpy="${0.00000 * deg_to_rad} ${0.00000 * deg_to_rad} ${0.00000 * deg_to_rad}"/>
+      <origin xyz="${0.00000 + head_2_joint_x_offset} ${0.00000 + head_2_joint_y_offset} ${0.00000 + head_2_joint_z_offset}"
+              rpy="${0.00000 * deg_to_rad + head_2_joint_roll_offset} ${0.00000 * deg_to_rad + head_2_joint_pitch_offset} ${0.00000 * deg_to_rad + head_2_joint_yaw_offset}"/>
       <axis xyz="0 0 1" />
       <limit lower="${-75.00000 * deg_to_rad}" upper="${75.00000 * deg_to_rad}" effort="4.0" velocity="${head_max_vel}" />

File: talos_description/urdf/torso/torso.urdf.xacro (robot description, xacro)
@@ -60,6 +60,6 @@
       <child link="${name}_1_link"/>
       <!-- XXX AS: The kinematic chain order for the torso was reversed manually. This value does not match the CAD model. XXX -->
-      <origin xyz="0.0 0.0 0.0722"
-              rpy="${0.00000 * deg_to_rad} ${0.00000 * deg_to_rad} ${0.00000 * deg_to_rad}"/>
+      <origin xyz="${0.0 + torso_1_joint_x_offset} ${0.0 + torso_1_joint_y_offset} ${0.0722 + torso_1_joint_z_offset}"
+              rpy="${0.00000 * deg_to_rad + torso_1_joint_roll_offset} ${0.00000 * deg_to_rad + torso_1_joint_pitch_offset} ${0.00000 * deg_to_rad + torso_1_joint_yaw_offset}"/>
       <axis xyz="0 0 1" />
       <limit lower="${-72.00000 * deg_to_rad}" upper="${72.00000 * deg_to_rad}"
@@ -93,6 +93,6 @@
       <parent link="${name}_1_link"/>
       <child link="${name}_2_link"/>
-      <origin xyz="0.0 0.0 0.0"
-              rpy="${0.00000 * deg_to_rad} ${0.00000 * deg_to_rad} ${0.00000 * deg_to_rad}"/>
+      <origin xyz="${0.0 + torso_1_joint_x_offset} ${0.0 + torso_1_joint_y_offset} ${0.0 + torso_1_joint_z_offset}"
+              rpy="${0.00000 * deg_to_rad + torso_1_joint_roll_offset} ${0.00000 * deg_to_rad + torso_1_joint_pitch_offset} ${0.00000 * deg_to_rad + torso_1_joint_yaw_offset}"/>
       <axis xyz="0 1 0" />
       <limit lower="${-13.0 * deg_to_rad}" upper="${42.0 * deg_to_rad}"

File: talos_description_calibration/urdf/calibration/calibration_constants.urdf.xacro (robot description, xacro)
@@ -33,4 +33,28 @@
   <xacro:property name="head_1_joint_offset" value="0.0" />
   <xacro:property name="head_2_joint_offset" value="0.0" />
+  <xacro:property name="head_1_joint_x_offset"     value="0.0" />
+  <xacro:property name="head_1_joint_y_offset"     value="0.0" />
+  <xacro:property name="head_1_joint_z_offset"     value="0.0" />
+  <xacro:property name="head_1_joint_roll_offset"  value="0.0" />
+  <xacro:property name="head_1_joint_pitch_offset" value="0.0" />
+  <xacro:property name="head_1_joint_yaw_offset"   value="0.0" />
+  <xacro:property name="head_2_joint_x_offset"     value="0.0" />
+  <xacro:property name="head_2_joint_y_offset"     value="0.0" />
+  <xacro:property name="head_2_joint_z_offset"     value="0.0" />
+  <xacro:property name="head_2_joint_roll_offset"  value="0.0" />
+  <xacro:property name="head_2_joint_pitch_offset" value="0.0" />
+  <xacro:property name="head_2_joint_yaw_offset"   value="0.0" />
+  <xacro:property name="torso_1_joint_x_offset"     value="0.0" />
+  <xacro:property name="torso_1_joint_y_offset"     value="0.0" />
+  <xacro:property name="torso_1_joint_z_offset"     value="0.0" />
+  <xacro:property name="torso_1_joint_roll_offset"  value="0.0" />
+  <xacro:property name="torso_1_joint_pitch_offset" value="0.0" />
+  <xacro:property name="torso_1_joint_yaw_offset"   value="0.0" />
+  <xacro:property name="torso_2_joint_x_offset"     value="0.0" />
+  <xacro:property name="torso_2_joint_y_offset"     value="0.0" />
+  <xacro:property name="torso_2_joint_z_offset"     value="0.0" />
+  <xacro:property name="torso_2_joint_roll_offset"  value="0.0" />
+  <xacro:property name="torso_2_joint_pitch_offset" value="0.0" />
+  <xacro:property name="torso_2_joint_yaw_offset"   value="0.0" />
   <xacro:property name="torso_imu_x_offset" value="0.0" />
   <xacro:property name="torso_imu_y_offset" value="0.0" />
