Commit message: [WIP] Add calibration file for Pyrene.

File: talos_description_calibration/urdf/calibration/arm_left.xacro (robot description, xacro)
@@ -1,52 +1,53 @@
-<?xml version="1.0"?>
-<!--
-  Copyright (c) 2015, PAL Robotics, S.L.
-  All rights reserved.
-  This work is licensed under the Creative Commons Attribution-NonCommercial-NoDerivs 3.0 Unported License.
-  To view a copy of this license, visit http://creativecommons.org/licenses/by-nc-nd/3.0/ or send a letter to
-  Creative Commons, 444 Castro Street, Suite 900, Mountain View, California, 94041, USA.
--->
+<?xml version='1.0' encoding='UTF-8'?>
+<!-- This file was generated automatically by package talos_calibration. -->
 <robot xmlns:xacro="http://ros.org/wiki/xacro">
-  <xacro:property name="arm_1_joint_x_offset"     value="0.0" />
-  <xacro:property name="arm_1_joint_y_offset"     value="0.0" />
-  <xacro:property name="arm_1_joint_z_offset"     value="0.0" />
-  <xacro:property name="arm_1_joint_roll_offset"  value="0.0" />
-  <xacro:property name="arm_1_joint_pitch_offset" value="0.0" />
-  <xacro:property name="arm_1_joint_yaw_offset"   value="0.0" />
-  <xacro:property name="arm_2_joint_x_offset"     value="0.0" />
-  <xacro:property name="arm_2_joint_y_offset"     value="0.0" />
-  <xacro:property name="arm_2_joint_z_offset"     value="0.0" />
-  <xacro:property name="arm_2_joint_roll_offset"  value="0.0" />
-  <xacro:property name="arm_2_joint_pitch_offset" value="0.0" />
-  <xacro:property name="arm_2_joint_yaw_offset"   value="0.0" />
-  <xacro:property name="arm_3_joint_x_offset"     value="0.0" />
-  <xacro:property name="arm_3_joint_y_offset"     value="0.0" />
-  <xacro:property name="arm_3_joint_z_offset"     value="0.0" />
-  <xacro:property name="arm_3_joint_roll_offset"  value="0.0" />
-  <xacro:property name="arm_3_joint_pitch_offset" value="0.0" />
-  <xacro:property name="arm_3_joint_yaw_offset"   value="0.0" />
-  <xacro:property name="arm_4_joint_x_offset"     value="0.0" />
-  <xacro:property name="arm_4_joint_y_offset"     value="0.0" />
-  <xacro:property name="arm_4_joint_z_offset"     value="0.0" />
-  <xacro:property name="arm_4_joint_roll_offset"  value="0.0" />
-  <xacro:property name="arm_4_joint_pitch_offset" value="0.0" />
-  <xacro:property name="arm_4_joint_yaw_offset"   value="0.0" />
-  <xacro:property name="arm_5_joint_x_offset"     value="0.0" />
-  <xacro:property name="arm_5_joint_y_offset"     value="0.0" />
-  <xacro:property name="arm_5_joint_z_offset"     value="0.0" />
-  <xacro:property name="arm_5_joint_roll_offset"  value="0.0" />
-  <xacro:property name="arm_5_joint_pitch_offset" value="0.0" />
-  <xacro:property name="arm_5_joint_yaw_offset"   value="0.0" />
-  <xacro:property name="arm_6_joint_x_offset"     value="0.0" />
-  <xacro:property name="arm_6_joint_y_offset"     value="0.0" />
-  <xacro:property name="arm_6_joint_z_offset"     value="0.0" />
-  <xacro:property name="arm_6_joint_roll_offset"  value="0.0" />
-  <xacro:property name="arm_6_joint_pitch_offset" value="0.0" />
-  <xacro:property name="arm_6_joint_yaw_offset"   value="0.0" />
-  <xacro:property name="arm_7_joint_x_offset"     value="0.0" />
-  <xacro:property name="arm_7_joint_y_offset"     value="0.0" />
-  <xacro:property name="arm_7_joint_z_offset"     value="0.0" />
-  <xacro:property name="arm_7_joint_roll_offset"  value="0.0" />
-  <xacro:property name="arm_7_joint_pitch_offset" value="0.0" />
-  <xacro:property name="arm_7_joint_yaw_offset"   value="0.0" />
+  <!--
+    Offsets in this file are such that `CAO + offset = reality`.
+    Unless stated otherwise, angles are in radians.
+    -->
+  <!--File includes-->
+  <xacro:include filename="$(find talos_description_calibration)/urdf/deg_to_rad.xacro"/>
+  <!--Constant parameters-->
+  <xacro:property name="arm_left_1_joint_x_offset" value="1.763e-05"/>
+  <xacro:property name="arm_left_1_joint_y_offset" value="-0.0014705"/>
+  <xacro:property name="arm_left_1_joint_z_offset" value="0.0013202"/>
+  <xacro:property name="arm_left_1_joint_yaw_offset" value="-0.0012607"/>
+  <xacro:property name="arm_left_1_joint_pitch_offset" value="0.0086499"/>
+  <xacro:property name="arm_left_1_joint_roll_offset" value="-0.022558"/>
+  <xacro:property name="arm_left_2_joint_x_offset" value="-0.0035031"/>
+  <xacro:property name="arm_left_2_joint_y_offset" value="-0.0014641"/>
+  <xacro:property name="arm_left_2_joint_z_offset" value="0.0024729"/>
+  <xacro:property name="arm_left_2_joint_yaw_offset" value="-0.022125"/>
+  <xacro:property name="arm_left_2_joint_pitch_offset" value="0.0086501"/>
+  <xacro:property name="arm_left_2_joint_roll_offset" value="-0.022667"/>
+  <xacro:property name="arm_left_3_joint_x_offset" value="-0.0034806"/>
+  <xacro:property name="arm_left_3_joint_y_offset" value="-0.0015782"/>
+  <xacro:property name="arm_left_3_joint_z_offset" value="0.00056011"/>
+  <xacro:property name="arm_left_3_joint_yaw_offset" value="-0.022255"/>
+  <xacro:property name="arm_left_3_joint_pitch_offset" value="0.010112"/>
+  <xacro:property name="arm_left_3_joint_roll_offset" value="-0.010015"/>
+  <xacro:property name="arm_left_4_joint_x_offset" value="-0.0014512"/>
+  <xacro:property name="arm_left_4_joint_y_offset" value="0.004296"/>
+  <xacro:property name="arm_left_4_joint_z_offset" value="0.00082743"/>
+  <xacro:property name="arm_left_4_joint_yaw_offset" value="-0.022949"/>
+  <xacro:property name="arm_left_4_joint_pitch_offset" value="0.003591"/>
+  <xacro:property name="arm_left_4_joint_roll_offset" value="-0.010165"/>
+  <xacro:property name="arm_left_5_joint_x_offset" value="-0.0021549"/>
+  <xacro:property name="arm_left_5_joint_y_offset" value="0.010119"/>
+  <xacro:property name="arm_left_5_joint_z_offset" value="0.0028305"/>
+  <xacro:property name="arm_left_5_joint_yaw_offset" value="-0.023012"/>
+  <xacro:property name="arm_left_5_joint_pitch_offset" value="0.0035377"/>
+  <xacro:property name="arm_left_5_joint_roll_offset" value="-0.0078481"/>
+  <xacro:property name="arm_left_6_joint_x_offset" value="-0.00072238"/>
+  <xacro:property name="arm_left_6_joint_y_offset" value="0.010535"/>
+  <xacro:property name="arm_left_6_joint_z_offset" value="0.0028454"/>
+  <xacro:property name="arm_left_6_joint_yaw_offset" value="-0.020495"/>
+  <xacro:property name="arm_left_6_joint_pitch_offset" value="0.0038764"/>
+  <xacro:property name="arm_left_6_joint_roll_offset" value="-0.0078403"/>
+  <xacro:property name="arm_left_7_joint_x_offset" value="-0.00071354"/>
+  <xacro:property name="arm_left_7_joint_y_offset" value="0.010584"/>
+  <xacro:property name="arm_left_7_joint_z_offset" value="0.00046582"/>
+  <xacro:property name="arm_left_7_joint_yaw_offset" value="-0.020494"/>
+  <xacro:property name="arm_left_7_joint_pitch_offset" value="0.0038818"/>
+  <xacro:property name="arm_left_7_joint_roll_offset" value="-0.0081044"/>
 </robot>

File: talos_description_calibration/urdf/calibration/arm_right.xacro (robot description, xacro)
@@ -1,52 +1,53 @@
-<?xml version="1.0"?>
-<!--
-  Copyright (c) 2015, PAL Robotics, S.L.
-  All rights reserved.
-  This work is licensed under the Creative Commons Attribution-NonCommercial-NoDerivs 3.0 Unported License.
-  To view a copy of this license, visit http://creativecommons.org/licenses/by-nc-nd/3.0/ or send a letter to
-  Creative Commons, 444 Castro Street, Suite 900, Mountain View, California, 94041, USA.
--->
+<?xml version='1.0' encoding='UTF-8'?>
+<!-- This file was generated automatically by package talos_calibration. -->
 <robot xmlns:xacro="http://ros.org/wiki/xacro">
-  <xacro:property name="arm_1_joint_x_offset"     value="0.0" />
-  <xacro:property name="arm_1_joint_y_offset"     value="0.0" />
-  <xacro:property name="arm_1_joint_z_offset"     value="0.0" />
-  <xacro:property name="arm_1_joint_roll_offset"  value="0.0" />
-  <xacro:property name="arm_1_joint_pitch_offset" value="0.0" />
-  <xacro:property name="arm_1_joint_yaw_offset"   value="0.0" />
-  <xacro:property name="arm_2_joint_x_offset"     value="0.0" />
-  <xacro:property name="arm_2_joint_y_offset"     value="0.0" />
-  <xacro:property name="arm_2_joint_z_offset"     value="0.0" />
-  <xacro:property name="arm_2_joint_roll_offset"  value="0.0" />
-  <xacro:property name="arm_2_joint_pitch_offset" value="0.0" />
-  <xacro:property name="arm_2_joint_yaw_offset"   value="0.0" />
-  <xacro:property name="arm_3_joint_x_offset"     value="0.0" />
-  <xacro:property name="arm_3_joint_y_offset"     value="0.0" />
-  <xacro:property name="arm_3_joint_z_offset"     value="0.0" />
-  <xacro:property name="arm_3_joint_roll_offset"  value="0.0" />
-  <xacro:property name="arm_3_joint_pitch_offset" value="0.0" />
-  <xacro:property name="arm_3_joint_yaw_offset"   value="0.0" />
-  <xacro:property name="arm_4_joint_x_offset"     value="0.0" />
-  <xacro:property name="arm_4_joint_y_offset"     value="0.0" />
-  <xacro:property name="arm_4_joint_z_offset"     value="0.0" />
-  <xacro:property name="arm_4_joint_roll_offset"  value="0.0" />
-  <xacro:property name="arm_4_joint_pitch_offset" value="0.0" />
-  <xacro:property name="arm_4_joint_yaw_offset"   value="0.0" />
-  <xacro:property name="arm_5_joint_x_offset"     value="0.0" />
-  <xacro:property name="arm_5_joint_y_offset"     value="0.0" />
-  <xacro:property name="arm_5_joint_z_offset"     value="0.0" />
-  <xacro:property name="arm_5_joint_roll_offset"  value="0.0" />
-  <xacro:property name="arm_5_joint_pitch_offset" value="0.0" />
-  <xacro:property name="arm_5_joint_yaw_offset"   value="0.0" />
-  <xacro:property name="arm_6_joint_x_offset"     value="0.0" />
-  <xacro:property name="arm_6_joint_y_offset"     value="0.0" />
-  <xacro:property name="arm_6_joint_z_offset"     value="0.0" />
-  <xacro:property name="arm_6_joint_roll_offset"  value="0.0" />
-  <xacro:property name="arm_6_joint_pitch_offset" value="0.0" />
-  <xacro:property name="arm_6_joint_yaw_offset"   value="0.0" />
-  <xacro:property name="arm_7_joint_x_offset"     value="0.0" />
-  <xacro:property name="arm_7_joint_y_offset"     value="0.0" />
-  <xacro:property name="arm_7_joint_z_offset"     value="0.0" />
-  <xacro:property name="arm_7_joint_roll_offset"  value="0.0" />
-  <xacro:property name="arm_7_joint_pitch_offset" value="0.0" />
-  <xacro:property name="arm_7_joint_yaw_offset"   value="0.0" />
+  <!--
+    Offsets in this file are such that `CAO + offset = reality`.
+    Unless stated otherwise, angles are in radians.
+    -->
+  <!--File includes-->
+  <xacro:include filename="$(find talos_description_calibration)/urdf/deg_to_rad.xacro"/>
+  <!--Constant parameters-->
+  <xacro:property name="arm_right_1_joint_x_offset" value="-0.0027269"/>
+  <xacro:property name="arm_right_1_joint_y_offset" value="-0.0023989"/>
+  <xacro:property name="arm_right_1_joint_z_offset" value="0.0018018"/>
+  <xacro:property name="arm_right_1_joint_yaw_offset" value="-0.0055284"/>
+  <xacro:property name="arm_right_1_joint_pitch_offset" value="0.0085537"/>
+  <xacro:property name="arm_right_1_joint_roll_offset" value="0.011974"/>
+  <xacro:property name="arm_right_2_joint_x_offset" value="-0.0041624"/>
+  <xacro:property name="arm_right_2_joint_y_offset" value="-0.0027134"/>
+  <xacro:property name="arm_right_2_joint_z_offset" value="0.0022602"/>
+  <xacro:property name="arm_right_2_joint_yaw_offset" value="0.0081435"/>
+  <xacro:property name="arm_right_2_joint_pitch_offset" value="0.0085524"/>
+  <xacro:property name="arm_right_2_joint_roll_offset" value="0.012216"/>
+  <xacro:property name="arm_right_3_joint_x_offset" value="-0.0041348"/>
+  <xacro:property name="arm_right_3_joint_y_offset" value="-0.0027875"/>
+  <xacro:property name="arm_right_3_joint_z_offset" value="-0.00087642"/>
+  <xacro:property name="arm_right_3_joint_yaw_offset" value="0.008148"/>
+  <xacro:property name="arm_right_3_joint_pitch_offset" value="0.0090689"/>
+  <xacro:property name="arm_right_3_joint_roll_offset" value="0.011728"/>
+  <xacro:property name="arm_right_4_joint_x_offset" value="-0.0023047"/>
+  <xacro:property name="arm_right_4_joint_y_offset" value="-0.0046688"/>
+  <xacro:property name="arm_right_4_joint_z_offset" value="-0.00068469"/>
+  <xacro:property name="arm_right_4_joint_yaw_offset" value="0.007134"/>
+  <xacro:property name="arm_right_4_joint_pitch_offset" value="0.033023"/>
+  <xacro:property name="arm_right_4_joint_roll_offset" value="0.011557"/>
+  <xacro:property name="arm_right_5_joint_x_offset" value="0.0049976"/>
+  <xacro:property name="arm_right_5_joint_y_offset" value="-0.0063257"/>
+  <xacro:property name="arm_right_5_joint_z_offset" value="-0.00078884"/>
+  <xacro:property name="arm_right_5_joint_yaw_offset" value="0.0072901"/>
+  <xacro:property name="arm_right_5_joint_pitch_offset" value="0.032926"/>
+  <xacro:property name="arm_right_5_joint_roll_offset" value="-0.0022284"/>
+  <xacro:property name="arm_right_6_joint_x_offset" value="0.0049478"/>
+  <xacro:property name="arm_right_6_joint_y_offset" value="-0.0062115"/>
+  <xacro:property name="arm_right_6_joint_z_offset" value="-0.00079128"/>
+  <xacro:property name="arm_right_6_joint_yaw_offset" value="0.0061621"/>
+  <xacro:property name="arm_right_6_joint_pitch_offset" value="0.032431"/>
+  <xacro:property name="arm_right_6_joint_roll_offset" value="-0.0022248"/>
+  <xacro:property name="arm_right_7_joint_x_offset" value="0.0049804"/>
+  <xacro:property name="arm_right_7_joint_y_offset" value="-0.0062177"/>
+  <xacro:property name="arm_right_7_joint_z_offset" value="-0.0017958"/>
+  <xacro:property name="arm_right_7_joint_yaw_offset" value="0.0061663"/>
+  <xacro:property name="arm_right_7_joint_pitch_offset" value="0.03243"/>
+  <xacro:property name="arm_right_7_joint_roll_offset" value="-0.0023539"/>
 </robot>

File: talos_description_calibration/urdf/calibration/calibration_constants.urdf.xacro (robot description, xacro)
@@ -1,14 +1,13 @@
-<?xml version="1.0"?>
-<!--
-  Copyright (c) 2015, PAL Robotics, S.L.
-  All rights reserved.
-  This work is licensed under the Creative Commons Attribution-NonCommercial-NoDerivs 3.0 Unported License.
-  To view a copy of this license, visit http://creativecommons.org/licenses/by-nc-nd/3.0/ or send a letter to
-  Creative Commons, 444 Castro Street, Suite 900, Mountain View, California, 94041, USA.
--->
+<?xml version='1.0' encoding='UTF-8'?>
+<!-- This file was generated automatically by package talos_calibration. -->
 <robot xmlns:xacro="http://ros.org/wiki/xacro">
+  <!--
+    Offsets in this file are such that `CAO + offset = reality`.
+    Unless stated otherwise, angles are in radians.
+    -->
   <!--File includes-->
   <xacro:include filename="$(find talos_description_calibration)/urdf/deg_to_rad.xacro" />
   <!--Constant parameters-->
+  <!-- Camera position (rgbd_joint wrt head_2_link) -->
   <xacro:property name="camera_position_x" value="0.066" />
   <xacro:property name="camera_position_y" value="0.0" />
@@ -33,34 +32,35 @@
   <xacro:property name="head_1_joint_offset" value="0.0" />
   <xacro:property name="head_2_joint_offset" value="0.0" />
-  <xacro:property name="head_1_joint_x_offset"     value="0.0" />
-  <xacro:property name="head_1_joint_y_offset"     value="0.0" />
-  <xacro:property name="head_1_joint_z_offset"     value="0.0" />
-  <xacro:property name="head_1_joint_roll_offset"  value="0.0" />
+  <xacro:property name="head_1_joint_x_offset" value="0.0" />
+  <xacro:property name="head_1_joint_y_offset" value="0.0" />
+  <xacro:property name="head_1_joint_z_offset" value="0.0" />
+  <xacro:property name="head_1_joint_roll_offset" value="0.0" />
   <xacro:property name="head_1_joint_pitch_offset" value="0.0" />
-  <xacro:property name="head_1_joint_yaw_offset"   value="0.0" />
-  <xacro:property name="head_2_joint_x_offset"     value="0.0" />
-  <xacro:property name="head_2_joint_y_offset"     value="0.0" />
-  <xacro:property name="head_2_joint_z_offset"     value="0.0" />
-  <xacro:property name="head_2_joint_roll_offset"  value="0.0" />
-  <xacro:property name="head_2_joint_pitch_offset" value="0.0" />
-  <xacro:property name="head_2_joint_yaw_offset"   value="0.0" />
-  <xacro:property name="torso_1_joint_x_offset"     value="0.0" />
-  <xacro:property name="torso_1_joint_y_offset"     value="0.0" />
-  <xacro:property name="torso_1_joint_z_offset"     value="0.0" />
-  <xacro:property name="torso_1_joint_roll_offset"  value="0.0" />
+  <xacro:property name="head_1_joint_yaw_offset" value="0.0" />
+  <xacro:property name="head_2_joint_x_offset" value="0.0018431" />
+  <xacro:property name="head_2_joint_y_offset" value="-0.0011307" />
+  <xacro:property name="head_2_joint_z_offset" value="5.9768e-07" />
+  <xacro:property name="head_2_joint_roll_offset" value="0.0005286" />
+  <xacro:property name="head_2_joint_pitch_offset" value="0.0086193" />
+  <xacro:property name="head_2_joint_yaw_offset" value="-4.5561e-06" />
+  <xacro:property name="torso_1_joint_x_offset" value="0.0" />
+  <xacro:property name="torso_1_joint_y_offset" value="0.0" />
+  <xacro:property name="torso_1_joint_z_offset" value="0.0" />
+  <xacro:property name="torso_1_joint_roll_offset" value="0.0" />
   <xacro:property name="torso_1_joint_pitch_offset" value="0.0" />
-  <xacro:property name="torso_1_joint_yaw_offset"   value="0.0" />
-  <xacro:property name="torso_2_joint_x_offset"     value="0.0" />
-  <xacro:property name="torso_2_joint_y_offset"     value="0.0" />
-  <xacro:property name="torso_2_joint_z_offset"     value="0.0" />
-  <xacro:property name="torso_2_joint_roll_offset"  value="0.0" />
-  <xacro:property name="torso_2_joint_pitch_offset" value="0.0" />
-  <xacro:property name="torso_2_joint_yaw_offset"   value="0.0" />
-  <xacro:property name="torso_imu_x_offset" value="0.0" />
-  <xacro:property name="torso_imu_y_offset" value="0.0" />
-  <xacro:property name="torso_imu_z_offset" value="0.0" />
+  <xacro:property name="torso_1_joint_yaw_offset" value="0.0" />
+  <xacro:property name="torso_2_joint_x_offset" value="0.0018431" />
+  <xacro:property name="torso_2_joint_y_offset" value="-0.0011307" />
+  <xacro:property name="torso_2_joint_z_offset" value="5.9768e-07" />
+  <xacro:property name="torso_2_joint_roll_offset" value="0.0005286" />
+  <xacro:property name="torso_2_joint_pitch_offset" value="0.0086193" />
+  <xacro:property name="torso_2_joint_yaw_offset" value="-4.5561e-06" />
+  <!-- IMU position offsets -->
+  <xacro:property name="torso_imu_x_offset" value="0." />
+  <xacro:property name="torso_imu_y_offset" value="0." />
+  <xacro:property name="torso_imu_z_offset" value="0." />
   <!-- Torso rpy offsets in degrees -->
-  <xacro:property name="torso_imu_roll_offset" value="0.0" />
-  <xacro:property name="torso_imu_pitch_offset" value="0.0" />
-  <xacro:property name="torso_imu_yaw_offset" value="0.0" />
+  <xacro:property name="torso_imu_roll_offset" value="0." />
+  <xacro:property name="torso_imu_pitch_offset" value="0." />
+  <xacro:property name="torso_imu_yaw_offset" value="0." />
 </robot>
